Commit message: added base extension layer and realsense d435 depth cam

File: betabot_description/urdf/betabot.gazebo.xacro (robot description, xacro)
@@ -7,5 +7,5 @@
   | |_/ /|  __/| |_ | (_| || |_) || (_) || |_
   \____/  \___| \__| \__,_||_.__/  \___/  \__| Gazebo Plugins-->
-<robot>
+<robot name="betabot_gazebo" xmlns:xacro="http://ros.org/wiki/xacro">
   <!-- <gazebo reference="left_wheel_link">
     <mu1>0.1</mu1>
@@ -43,5 +43,5 @@
   </gazebo> -->
 <!-- ***** RASPBERRY PI 8MB CAMERA SIMULATED ***** -->
-  <gazebo reference="camera_link">
+  <!--gazebo reference="camera_link">
     <sensor type="camera" name="camera">
       <update_rate>30.0</update_rate>
@@ -61,5 +61,5 @@
       <plugin name="camera_controller" filename="libgazebo_ros_camera.so">
         <updateRate>0.0</updateRate>
-        <cameraName>betabot/camera</cameraName>
+        <cameraName>/camera</cameraName>
         <imageTopicName>image_raw</imageTopicName>
         <cameraInfoTopicName>camera_info</cameraInfoTopicName>
@@ -73,10 +73,10 @@
       </plugin>
     </sensor>
-  </gazebo>
+  </gazebo-->
 <!-- ***** BETABOT DD CONTROLLER ***** -->
   <gazebo>
     <plugin name="differential_drive_controller" filename="libgazebo_ros_diff_drive.so">
-      <commandTopic>betabot/cmd_vel</commandTopic>
-      <odometryTopic>betabot/odom</odometryTopic>
+      <commandTopic>/cmd_vel</commandTopic>
+      <odometryTopic>/odom</odometryTopic>
       <odometryFrame>odom</odometryFrame>
       <odometrySource>world</odometrySource>
@@ -87,5 +87,5 @@
       <publishWheelJointState>true</publishWheelJointState>
       <legacyMode>false</legacyMode>
-      <updateRate>30</updateRate>
+      <updateRate>60</updateRate>
       <leftJoint>left_wheel_joint</leftJoint>
       <rightJoint>right_wheel_joint</rightJoint>
@@ -93,24 +93,14 @@
       <wheelDiameter>0.065</wheelDiameter>
       <wheelAcceleration>1</wheelAcceleration>
-      <wheelTorque>10</wheelTorque>
+      <wheelTorque>5</wheelTorque>
       <rosDebugLevel>na</rosDebugLevel>
     </plugin>
   </gazebo>
-<!-- UNCOMMENT TO FORCE SPECIFIC MESH COLOR FOR BETABOT PARTS  -->
-  <!-- <gazebo reference="base_link">
-    <material>Gazebo/Orange</material>
-  </gazebo>
-  <gazebo reference="left_wheel">
-    <material>Gazebo/Blue</material>
-  </gazebo>
-  <gazebo reference="right_wheel">
-    <material>Gazebo/Blue</material>
-  </gazebo> -->
-  <!-- hokuyo -->
+  <!-- Rplidar -->
   <gazebo reference="rplidar_link">
     <sensor type="gpu_ray" name="head_hokuyo_sensor">
       <pose>0 0 0 0 0 0</pose>
       <visualize>false</visualize>
-      <update_rate>40</update_rate>
+      <update_rate>100</update_rate>
       <ray>
         <scan>
@@ -138,9 +128,10 @@
       </ray>
       <plugin name="gazebo_ros_head_rplidar_controller" filename="libgazebo_ros_gpu_laser.so">
-        <topicName>betabot/laser/scan</topicName>
+        <topicName>/scan</topicName>
         <frameName>rplidar_link</frameName>
       </plugin>
     </sensor>
   </gazebo>
+  <!-- Realsense d435 -->
   <gazebo>
     <plugin name="imu_plugin" filename="libgazebo_ros_imu.so">
@@ -151,5 +142,5 @@
       <serviceName>imu_service</serviceName>
       <gaussianNoise>0.0</gaussianNoise>
-      <updateRate>200</updateRate>
+      <updateRate>60</updateRate>
       <imu>
         <noise>
@@ -171,3 +162,39 @@
     </plugin>
   </gazebo>
+  <gazebo reference="camera_link">
+    <sensor type="depth" name="camera">
+      <always_on>true</always_on>
+      <update_rate>20.0</update_rate>
+      <camera>
+        <horizontal_fov>${86.0*M_PI/180.0}</horizontal_fov>
+        <image>
+          <format>B8G8R8</format>
+          <width>640</width>
+          <height>480</height>
+        </image>
+        <clip>
+          <near>0.02</near>
+          <far>8.0</far>
+        </clip>
+      </camera>
+      <plugin name="kinect_camera_controller" filename="libgazebo_ros_openni_kinect.so">
+        <cameraName>camera</cameraName>
+        <alwaysOn>true</alwaysOn>
+        <updateRate>10</updateRate>
+        <imageTopicName>rgb/image_raw</imageTopicName>
+        <depthImageTopicName>depth/image_raw</depthImageTopicName>
+        <pointCloudTopicName>depth/points</pointCloudTopicName>
+        <cameraInfoTopicName>rgb/camera_info</cameraInfoTopicName>
+        <depthImageCameraInfoTopicName>depth/camera_info</depthImageCameraInfoTopicName>
+        <frameName>camera_depth_optical_frame</frameName>
+        <baseline>0.1</baseline>
+        <distortion_k1>0.0</distortion_k1>
+        <distortion_k2>0.0</distortion_k2>
+        <distortion_k3>0.0</distortion_k3>
+        <distortion_t1>0.0</distortion_t1>
+        <distortion_t2>0.0</distortion_t2>
+        <pointCloudCutoff>0.4</pointCloudCutoff>
+      </plugin>
+    </sensor>
+  </gazebo>
 </robot>

File: betabot_description/urdf/betabot.urdf.xacro (robot description, xacro)
@@ -6,10 +6,11 @@
   | ___ \ / _ \| __| / _` || '_ \  / _ \ | __|
   | |_/ /|  __/| |_ | (_| || |_) || (_) || |_
-  \____/  \___| \__| \__,_||_.__/  \___/  \__| URDF Description-->
+  \____/  \___| \__| \__,_||_.__/  \___/  \__| URDF-XACRO Description-->
 <robot name="betabot" xmlns:xacro="http://www.ros.org/wiki/xacro">
 <!-- CALL HEADER FILES FOR MACROS AND GAZEBO PLUGINS -->
   <xacro:include filename="$(find betabot_description)/urdf/betabot.gazebo.xacro" />
-  <xacro:include filename="$(find betabot_description)/urdf/materials.xacro" />
+  <xacro:include filename="$(find betabot_description)/urdf/common_properties.urdf.xacro" />
   <xacro:include filename="$(find betabot_description)/urdf/macros.xacro" />
+  <xacro:include filename="$(find betabot_description)/urdf/betabot_d435_properties.urdf.xacro" />
 <!-- ***** BETABOT BASE PART***** -->
   <link name="base_footprint"/>
@@ -206,7 +207,43 @@
     <axis xyz="0 0 0" />
   </joint>
+<!-- ***** BETABOT EXTENSION ***** -->
+  <joint name="base_extension_joint" type="fixed">
+    <parent link="base_link"/>
+    <child link="base_extension_link"/>
+    <origin xyz="0.0 0.0 0.35" rpy="0 0 0"/>
+  </joint>
+  <link name="base_extension_link">
+    <inertial>
+      <origin xyz="2.8456E-05 0.02785 0.00053742" rpy="0 0 0" />
+      <mass value="5.67773" />
+      <inertia ixx="0.019995" ixy="0.0" ixz="0.0" iyy="0.019995" iyz="0.0" izz="0.03675" />
+    </inertial>
+    <visual>
+      <origin xyz="0 0 0" rpy="0 0 1.5708" />
+      <geometry>
+        <mesh filename="package://betabot_description/meshes/betabot_extension.dae" />
+      </geometry>
+      <material name="">
+        <color rgba="0.79608 0.82353 0.93725 1" />
+      </material>
+    </visual>
+    <!-- COMMENT THE ORGINAL COLLISION MODEL,NEEDS MORE PROCESSING POWER -->
+    <!-- <collision>
+      <origin xyz="0 0 0" rpy="0 0 0" />
+      <geometry>
+        <mesh filename="package://betabot_description/meshes/betabot_base.dae" />
+      </geometry>
+    </collision> -->
+    <!-- SIMPLIFIED COLLISOION MESH FOR FOR SMOOTH PROCESSING -->
+    <collision>
+      <geometry>
+        <cylinder length="0.004" radius="0.15"/>
+      </geometry>
+      <origin rpy="0 0 0" xyz="0  0 0.05"/>
+    </collision>
+  </link>
 <!-- ***** RASPBERRY PI 8MB CAMERA SIMULATED PART ***** -->
   <!-- LINK -->
-  <link name="camera_link">
+  <!-- <link name="camera_link">
     <visual>
       <origin xyz="0 0 0" rpy="0 1.570 1.570" />
@@ -224,12 +261,12 @@
       <inertia ixx="1e-6" ixy="0" ixz="0" iyy="1e-6" iyz="0" izz="1e-6" />
     </inertial>
-  </link>
-  <!-- JOINT -->
-  <joint name="camera_joint" type="fixed">
+  </link> -->
+  <!-- JOINT -->
+  <!-- <joint name="camera_joint" type="fixed">
     <axis xyz="0 0 0" />
     <origin xyz="0.148 0 0.036" rpy="0 0 0"/>
     <parent link="base_link"/>
     <child link="camera_link"/>
-  </joint>
+  </joint>  -->
 <!-- ***** IMU SENSOR PART ***** -->
   <!-- LINK -->
@@ -312,7 +349,113 @@
   <joint name="rplidar_joint" type="fixed">
     <axis xyz="0 1 0" />
-    <origin xyz="0 0 .109" rpy="0 0 0"/>
+    <origin xyz="0 0 .109" rpy="0 0 1.57"/>
     <parent link="base_link"/>
     <child link="rplidar_link"/>
   </joint>
+<!-- REALSENSE SIMULATED PART -->
+<!-- URDF model for the Intel RealSense 430 camera, in it's aluminum peripherial evaluation case -->
+    <!--~~~~~~~~ camera body, with origin at bottom screw mount ~~~~~~~~-->
+    <!-- JOINT -->
+    <joint name="camera_joint" type="fixed">
+       <origin xyz="${cam_px} ${cam_py} ${cam_pz}" rpy="${cam_or} ${cam_op} ${cam_oy}"/>
+      <parent link="${parent}"/>
+      <child link="camera_bottom_screw_frame" />
+    </joint>
+    <link name="camera_bottom_screw_frame"/>
+    <joint name="camera_link_joint" type="fixed">
+      <origin xyz="0 ${d435_cam_depth_py} ${d435_cam_depth_pz}" rpy="0 0 0"/>
+      <parent link="camera_bottom_screw_frame"/>
+      <child link="camera_link" />
+    </joint>
+    <!-- LINK -->
+    <link name="camera_link">
+      <visual>
+      <origin xyz="${d435_cam_mount_from_center_offset} ${-d435_cam_depth_py} 0" rpy="${M_PI/2} 0 ${M_PI/2}"/>
+        <geometry>
+          <!-- <box size="${d435_cam_width} ${d435_cam_height} ${d435_cam_depth}"/> -->
+          <mesh filename="package://betabot_description/meshes/d435.dae" />
+          <!--<mesh filename="package://realsense2_description/meshes/d435/d435.dae" />-->
+        </geometry>
+      </visual>
+      <collision>
+        <origin xyz="0 ${-d435_cam_depth_py} 0" rpy="0 0 0"/>
+        <geometry>
+        <box size="${d435_cam_depth} ${d435_cam_width} ${d435_cam_height}"/>
+        </geometry>
+      </collision>
+      <inertial>
+        <!-- The following are not reliable values, and should not be used for modeling -->
+        <mass value="0.564" />
+        <origin xyz="0 0 0" />
+        <inertia ixx="0.003881243" ixy="0.0" ixz="0.0" iyy="0.000498940" iyz="0.0" izz="0.003879257" />
+      </inertial>
+    </link>
+    <!--~~~~~~~~ camera depth joints and links ~~~~~~~~-->
+    <!-- JOINT -->
+    <joint name="camera_depth_joint" type="fixed">
+      <origin xyz="0 0 0" rpy="0 0 0"/>
+      <parent link="camera_link"/>
+      <child link="camera_depth_frame" />
+    </joint>
+    <!-- LINK -->
+    <link name="camera_depth_frame"/>
+    <!-- JOINT -->
+    <joint name="camera_depth_optical_joint" type="fixed">
+      <origin xyz="0 0 0" rpy="${-M_PI/2} 0 ${-M_PI/2}" />
+      <parent link="camera_depth_frame" />
+      <child link="camera_depth_optical_frame" />
+    </joint>
+    <!-- LINK -->
+    <link name="camera_depth_optical_frame"/>
+    <!--~~~~~~~~ camera left IR joints and links ~~~~~~~~-->
+    <!-- JOINT -->
+    <joint name="camera_left_ir_joint" type="fixed">
+      <origin xyz="0 ${d435_cam_depth_to_left_ir_offset} 0" rpy="0 0 0" />
+      <parent link="camera_depth_frame" />
+      <child link="camera_left_ir_frame" />
+    </joint>
+    <!-- LINK -->
+    <link name="camera_left_ir_frame"/>
+    <!-- JOINT -->
+    <joint name="camera_left_ir_optical_joint" type="fixed">
+      <origin xyz="0 0 0" rpy="${-M_PI/2} 0 ${-M_PI/2}" />
+      <parent link="camera_left_ir_frame" />
+      <child link="camera_left_ir_optical_frame" />
+    </joint>
+    <!-- LINK -->
+    <link name="camera_left_ir_optical_frame"/>
+    <!--~~~~~~~~ camera right IR joints and links ~~~~~~~~-->
+    <!-- JOINT -->
+    <joint name="camera_right_ir_joint" type="fixed">
+      <origin xyz="0 ${d435_cam_depth_to_right_ir_offset} 0" rpy="0 0 0" />
+      <parent link="camera_depth_frame" />
+      <child link="camera_right_ir_frame" />
+    </joint>
+    <!-- LINK -->
+    <link name="camera_right_ir_frame"/>
+    <!-- JOINT -->
+    <joint name="camera_right_ir_optical_joint" type="fixed">
+      <origin xyz="0 0 0" rpy="${-M_PI/2} 0 ${-M_PI/2}" />
+      <parent link="camera_right_ir_frame" />
+      <child link="camera_right_ir_optical_frame" />
+    </joint>
+    <!-- LINK -->
+    <link name="camera_right_ir_optical_frame"/>
+    <!--~~~~~~~~ camera color joints and links ~~~~~~~~-->
+    <!-- JOINT -->
+    <joint name="camera_color_joint" type="fixed">
+      <origin xyz="0 ${d435_cam_depth_to_color_offset} 0" rpy="0 0 0" />
+      <parent link="camera_depth_frame" />
+      <child link="camera_color_frame" />
+    </joint>
+    <!-- LINK -->
+    <link name="camera_color_frame"/>
+    <!-- JOINT -->
+    <joint name="camera_color_optical_joint" type="fixed">
+      <origin xyz="0 0 0" rpy="${-M_PI/2} 0 ${-M_PI/2}" />
+      <parent link="camera_color_frame" />
+      <child link="camera_color_optical_frame" />
+    </joint>
+    <!-- LINK -->
+    <link name="camera_color_optical_frame"/>
 </robot>

Commit message: added friction

File: betabot_description/urdf/betabot.gazebo.xacro (robot description, xacro)
@@ -8,5 +8,7 @@
   \____/  \___| \__| \__,_||_.__/  \___/  \__| Gazebo Plugins-->
 <robot name="betabot_gazebo" xmlns:xacro="http://ros.org/wiki/xacro">
-  <!-- <gazebo reference="left_wheel_link">
+  <xacro:property name="M_PI" value="3.1415926535897931" />
+<!--
+  <gazebo reference="left_wheel_link">
     <mu1>0.1</mu1>
     <mu2>0.1</mu2>
@@ -41,4 +43,43 @@
     <minDepth>0.001</minDepth>
     <maxVel>1.0</maxVel>
+  </gazebo> -->
+<!--
+    <gazebo reference="left_wheel_link">
+    <mu1>0.1</mu1>
+    <mu2>0.1</mu2>
+    <kp>500000.0</kp>
+    <kd>10.0</kd>
+    <minDepth>0.001</minDepth>
+    <maxVel>0.1</maxVel>
+    <fdir1>1 0 0</fdir1>
+    <material>Gazebo/FlatBlack</material>
+  </gazebo>
+  <gazebo reference="right_wheel_link">
+    <mu1>0.1</mu1>
+    <mu2>0.1</mu2>
+    <kp>500000.0</kp>
+    <kd>10.0</kd>
+    <minDepth>0.001</minDepth>
+    <maxVel>0.1</maxVel>
+    <fdir1>1 0 0</fdir1>
+    <material>Gazebo/FlatBlack</material>
+  </gazebo>
+  <gazebo reference="back_caster_link">
+    <mu1>0.1</mu1>
+    <mu2>0.1</mu2>
+    <kp>1000000.0</kp>
+    <kd>100.0</kd>
+    <minDepth>0.001</minDepth>
+    <maxVel>1.0</maxVel>
+    <material>Gazebo/FlatBlack</material>
+  </gazebo>
+  <gazebo reference="front_caster_link">
+    <mu1>0.1</mu1>
+    <mu2>0.1</mu2>
+    <kp>1000000.0</kp>
+    <kd>100.0</kd>
+    <minDepth>0.001</minDepth>
+    <maxVel>1.0</maxVel>
+    <material>Gazebo/FlatBlack</material>
   </gazebo> -->
 <!-- ***** RASPBERRY PI 8MB CAMERA SIMULATED ***** -->

File: betabot_description/urdf/betabot.urdf.xacro (robot description, xacro)
@@ -13,4 +13,5 @@
   <xacro:include filename="$(find betabot_description)/urdf/macros.xacro" />
   <xacro:include filename="$(find betabot_description)/urdf/betabot_d435_properties.urdf.xacro" />
+  <xacro:property name="M_PI" value="3.1415926535897931" />
 <!-- ***** BETABOT BASE PART***** -->
   <link name="base_footprint"/>
@@ -85,4 +86,5 @@
     <child link="right_wheel_link" />
     <axis xyz="0 0 -1" />
+    <dynamics damping="0.1" friction="0.1"/>
   </joint>
 <!-- ***** BETABOT LEFT WHEEL PART ***** -->
@@ -125,4 +127,5 @@
     <child link="left_wheel_link" />
     <axis xyz="0 0 1" />
+    <dynamics damping="0.1" friction="0.1"/>
   </joint>
 <!-- ***** BETABOT FRONT CASTER WHEEL ***** -->

Commit message: added friction to wheels

File: betabot_description/urdf/betabot.gazebo.xacro (robot description, xacro)
@@ -9,22 +9,29 @@
 <robot name="betabot_gazebo" xmlns:xacro="http://ros.org/wiki/xacro">
   <xacro:property name="M_PI" value="3.1415926535897931" />
-<!--
-  <gazebo reference="left_wheel_link">
-    <mu1>0.1</mu1>
-    <mu2>0.1</mu2>
-    <kp>500000.0</kp>
-    <kd>10.0</kd>
-    <minDepth>0.001</minDepth>
-    <maxVel>0.1</maxVel>
-    <fdir1>0 1 0</fdir1>
+    <gazebo reference="left_wheel_link">
+    <mu1>0.1</mu1>
+    <mu2>0.1</mu2>
+    <kp>1000000000.0</kp>
+    <kd>100.0</kd>
+    <minDepth>0.001</minDepth>
+    <maxVel>1.0</maxVel>
+    <fdir1>1 0 0</fdir1>
   </gazebo>
   <gazebo reference="right_wheel_link">
     <mu1>0.1</mu1>
     <mu2>0.1</mu2>
-    <kp>500000.0</kp>
-    <kd>10.0</kd>
-    <minDepth>0.001</minDepth>
-    <maxVel>0.1</maxVel>
-    <fdir1>0 1 0</fdir1>
+    <kp>1000000000.0</kp>
+    <kd>100.0</kd>
+    <minDepth>0.001</minDepth>
+    <maxVel>1.0</maxVel>
+    <fdir1>1 0 0</fdir1>
+  </gazebo>
+  <gazebo reference="back_caster_link">
+    <mu1>0.1</mu1>
+    <mu2>0.1</mu2>
+    <kp>1000000.0</kp>
+    <kd>100.0</kd>
+    <minDepth>0.001</minDepth>
+    <maxVel>1.0</maxVel>
   </gazebo>
   <gazebo reference="front_caster_link">
@@ -36,51 +43,4 @@
     <maxVel>1.0</maxVel>
   </gazebo>
-  <gazebo reference="back_caster_link">
-    <mu1>0.1</mu1>
-    <mu2>0.1</mu2>
-    <kp>1000000.0</kp>
-    <kd>100.0</kd>
-    <minDepth>0.001</minDepth>
-    <maxVel>1.0</maxVel>
-  </gazebo> -->
-<!--
-    <gazebo reference="left_wheel_link">
-    <mu1>0.1</mu1>
-    <mu2>0.1</mu2>
-    <kp>500000.0</kp>
-    <kd>10.0</kd>
-    <minDepth>0.001</minDepth>
-    <maxVel>0.1</maxVel>
-    <fdir1>1 0 0</fdir1>
-    <material>Gazebo/FlatBlack</material>
-  </gazebo>
-  <gazebo reference="right_wheel_link">
-    <mu1>0.1</mu1>
-    <mu2>0.1</mu2>
-    <kp>500000.0</kp>
-    <kd>10.0</kd>
-    <minDepth>0.001</minDepth>
-    <maxVel>0.1</maxVel>
-    <fdir1>1 0 0</fdir1>
-    <material>Gazebo/FlatBlack</material>
-  </gazebo>
-  <gazebo reference="back_caster_link">
-    <mu1>0.1</mu1>
-    <mu2>0.1</mu2>
-    <kp>1000000.0</kp>
-    <kd>100.0</kd>
-    <minDepth>0.001</minDepth>
-    <maxVel>1.0</maxVel>
-    <material>Gazebo/FlatBlack</material>
-  </gazebo>
-  <gazebo reference="front_caster_link">
-    <mu1>0.1</mu1>
-    <mu2>0.1</mu2>
-    <kp>1000000.0</kp>
-    <kd>100.0</kd>
-    <minDepth>0.001</minDepth>
-    <maxVel>1.0</maxVel>
-    <material>Gazebo/FlatBlack</material>
-  </gazebo> -->
 <!-- ***** RASPBERRY PI 8MB CAMERA SIMULATED ***** -->
   <!--gazebo reference="camera_link">

File: betabot_description/urdf/betabot.urdf.xacro (robot description, xacro)
@@ -86,5 +86,4 @@
     <child link="right_wheel_link" />
     <axis xyz="0 0 -1" />
-    <dynamics damping="0.1" friction="0.1"/>
   </joint>
 <!-- ***** BETABOT LEFT WHEEL PART ***** -->
@@ -127,5 +126,4 @@
     <child link="left_wheel_link" />
     <axis xyz="0 0 1" />
-    <dynamics damping="0.1" friction="0.1"/>
   </joint>
 <!-- ***** BETABOT FRONT CASTER WHEEL ***** -->
@@ -168,4 +166,5 @@
     <child link="front_caster_link" />
     <axis xyz="0 0 0" />
+    <dynamics damping="0.0" friction="0.0"/>
   </joint>
 <!-- ***** BETABOT BACK CASTER WHEEL ***** -->
@@ -209,4 +208,5 @@
     <child link="back_caster_link" />
     <axis xyz="0 0 0" />
+    <dynamics damping="0.0" friction="0.0"/>
   </joint>
 <!-- ***** BETABOT EXTENSION ***** -->
