Commit message: modified physics

File: betabot_description/urdf/betabot.gazebo.xacro (robot description, xacro)
@@ -9,4 +9,5 @@
 <robot name="betabot_gazebo" xmlns:xacro="http://ros.org/wiki/xacro">
   <xacro:property name="M_PI" value="3.1415926535897931" />
+<!--
     <gazebo reference="left_wheel_link">
     <mu1>0.1</mu1>
@@ -42,5 +43,5 @@
     <minDepth>0.001</minDepth>
     <maxVel>1.0</maxVel>
-  </gazebo>
+  </gazebo> -->
 <!-- ***** RASPBERRY PI 8MB CAMERA SIMULATED ***** -->
   <!--gazebo reference="camera_link">

File: betabot_description/urdf/betabot.urdf.xacro (robot description, xacro)
@@ -19,9 +19,9 @@
     <parent link="base_footprint"/>
     <child link="base_link"/>
-    <origin xyz="0.0 0.0 0.010" rpy="0 0 0"/>
+    <origin xyz="0.0 0.0 0.01" rpy="0 0 0"/>
   </joint>
   <link name="base_link">
     <inertial>
-      <origin xyz="2.8456E-05 0.02785 0.00053742" rpy="0 0 0" />
+      <origin xyz="0 0 0" rpy="0 0 0"/>
       <mass value="5.67773" />
       <inertia ixx="0.019995" ixy="0.0" ixz="0.0" iyy="0.019995" iyz="0.0" izz="0.03675" />
@@ -54,7 +54,10 @@
   <link name="right_wheel_link">
     <inertial>
-      <origin xyz="1.7347E-17 -7.3726E-17 -0.015" rpy="0 0 0" />
-      <mass value="0.5" />
-      <inertia ixx="0.001" ixy="0.0" ixz="0.0" iyy="0.001" iyz="0.0" izz="0.001" />
+      <origin xyz="0 0 0" rpy="0 0 0"/>
+      <mass value="2"/>
+      <inertia
+        ixx=".08" ixy="0.0" ixz="0.0"
+        iyy=".08" iyz="0.0"
+        izz=".08"/>
     </inertial>
     <visual>
@@ -82,5 +85,5 @@
   <!-- JOINT -->
   <joint name="right_wheel_joint" type="continuous">
-    <origin xyz="0 -0.097 -0.0125" rpy="-1.5708 1.3735 3.14159265359" />
+    <origin xyz="0 -0.097 -0.0125" rpy="-1.57079632679 1.57079632679 3.14159265359" />
     <parent link="base_link" />
     <child link="right_wheel_link" />
@@ -91,7 +94,10 @@
   <link name="left_wheel_link">
     <inertial>
-      <origin xyz="-1.7347E-17 -7.3726E-17 -0.015" rpy="0 0 0" />
-      <mass value="0.5" />
-      <inertia ixx="0.001" ixy="0.0" ixz="0.0" iyy="0.001" iyz="0.0" izz="0.001" />
+      <origin xyz="0 0 0" rpy="0 0 0"/>
+      <mass value="2"/>
+      <inertia
+        ixx=".08" ixy="0.0" ixz="0.0"
+        iyy=".08" iyz="0.0"
+        izz=".08"/>
     </inertial>
     <visual>
@@ -122,5 +128,5 @@
   <!-- JOINT -->
   <joint name="left_wheel_joint" type="continuous">
-    <origin xyz="0 0.097 -0.0125" rpy="-1.5708 1.5228 0" />
+    <origin xyz="0 0.097 -0.0125" rpy="-1.57079632679 1.57079632679 0" />
     <parent link="base_link" />
     <child link="left_wheel_link" />
@@ -132,6 +138,8 @@
     <inertial>
       <origin xyz="0 -0.011704 0.02" rpy="0 0 0" />
-      <mass value="0.2" />
-      <inertia ixx="0.001" ixy="0.0" ixz="0.0" iyy="0.001" iyz="0.0"  izz="0.001" />
+      <mass value="0.005" />
+      <inertia ixx="0.001" ixy="0.0" ixz="0.0"
+               iyy="0.001" iyz="0.0"
+               izz="0.001" />
     </inertial>
     <visual>
@@ -157,14 +165,13 @@
          <sphere radius="0.020"/>
       </geometry>
-      <origin rpy="0 0 0" xyz="0 -0.0026 0"/>
+      <origin rpy="0 0 0" xyz="0 -0.0026 0.0"/>
     </collision>
   </link>
   <!-- JOINT -->
   <joint name="front_caster_joint" type="fixed">
-    <origin xyz="0.105 0 -0.02231" rpy="1.5708 6.123E-17 1.5708" />
+    <origin xyz="0.105 0 -0.02231" rpy="1.57079632679 0 1.57079632679" />
     <parent link="base_link" />
     <child link="front_caster_link" />
     <axis xyz="0 0 0" />
-    <dynamics damping="0.1" friction="0.1"/>
   </joint>
 <!-- ***** BETABOT BACK CASTER WHEEL ***** -->
@@ -173,6 +180,8 @@
     <inertial>
       <origin xyz="0 0.011704 0.02" rpy="0 0 0" />
-      <mass value="0.2" />
-      <inertia ixx="0.001" ixy="0.0" ixz="0.0" iyy="0.001" iyz="0.0" izz="0.001" />
+      <mass value="0.005" />
+      <inertia ixx="0.001" ixy="0.0" ixz="0.0"
+               iyy="0.001" iyz="0.0"
+               izz="0.001" />
     </inertial>
     <visual>
@@ -204,9 +213,8 @@
   <!-- JOINT -->
   <joint name="back_caster_joint" type="fixed">
-    <origin xyz="-0.105 0 -0.02231" rpy="1.5708 6.123E-17 1.5708" />
+    <origin xyz="-0.105 0 -0.02221" rpy="1.57079632679 0 1.57079632679" />
     <parent link="base_link" />
     <child link="back_caster_link" />
     <axis xyz="0 0 0" />
-    <dynamics damping="0.1" friction="0.1"/>
   </joint>
 <!-- ***** BETABOT EXTENSION ***** -->
@@ -219,5 +227,5 @@
     <inertial>
       <origin xyz="2.8456E-05 0.02785 0.00053742" rpy="0 0 0" />
-      <mass value="5.67773" />
+      <mass value="0.1" />
       <inertia ixx="0.019995" ixy="0.0" ixz="0.0" iyy="0.019995" iyz="0.0" izz="0.03675" />
     </inertial>
@@ -389,5 +397,5 @@
       <inertial>
         <!-- The following are not reliable values, and should not be used for modeling -->
-        <mass value="0.564" />
+        <mass value="0.01" />
         <origin xyz="0 0 0" />
         <inertia ixx="0.003881243" ixy="0.0" ixz="0.0" iyy="0.000498940" iyz="0.0" izz="0.003879257" />
