Commit message: clean and organize the package

File: betabot_description/urdf/betabot.urdf.xacro (robot description, xacro)
@@ -9,8 +9,14 @@
 <robot name="betabot" xmlns:xacro="http://www.ros.org/wiki/xacro">
 <!-- CALL HEADER FILES FOR MACROS AND GAZEBO PLUGINS -->
-  <xacro:include filename="$(find betabot)/betabot_description/urdf/betabot.gazebo" />
-  <xacro:include filename="$(find betabot)/betabot_description/urdf/materials.xacro" />
-  <xacro:include filename="$(find betabot)/betabot_description/urdf/macros.xacro" />
+  <xacro:include filename="$(find betabot_description)/urdf/betabot.gazebo" />
+  <xacro:include filename="$(find betabot_description)/urdf/materials.xacro" />
+  <xacro:include filename="$(find betabot_description)/urdf/macros.xacro" />
 <!-- ***** BETABOT BASE PART***** -->
+  <link name="base_footprint"/>
+  <joint name="base_joint" type="fixed">
+    <parent link="base_footprint"/>
+    <child link="base_link"/>
+    <origin xyz="0.0 0.0 0.010" rpy="0 0 0"/>
+  </joint>
   <link name="base_link">
     <inertial>
@@ -22,5 +28,5 @@
       <origin xyz="0 0 0" rpy="0 0 0" />
       <geometry>
-        <mesh filename="package://betabot/betabot_description/meshes/betabot_base.dae" />
+        <mesh filename="package://betabot_description/meshes/betabot_base.dae" />
       </geometry>
       <material name="">
@@ -32,5 +38,5 @@
       <origin xyz="0 0 0" rpy="0 0 0" />
       <geometry>
-        <mesh filename="package://betabot/betabot_description/meshes/betabot_base.dae" />
+        <mesh filename="package://betabot_description/meshes/betabot_base.dae" />
       </geometry>
     </collision> -->
@@ -53,5 +59,5 @@
       <origin xyz="0 0 0" rpy="0 0 0" />
       <geometry>
-        <mesh filename="package://betabot/betabot_description/meshes/betabot_wheel.dae" />
+        <mesh filename="package://betabot_description/meshes/betabot_wheel.dae" />
       </geometry>
       <material name="">
@@ -62,5 +68,5 @@
       <origin xyz="0 0 0" rpy="0 0 0" />
       <geometry>
-        <mesh filename="package://betabot/betabot_description/meshes/betabot_wheel.dae" />
+        <mesh filename="package://betabot_description/meshes/betabot_wheel.dae" />
       </geometry>
     </collision> -->
@@ -90,5 +96,5 @@
       <origin xyz="0 0 0" rpy="0 0 0" />
       <geometry>
-        <mesh filename="package://betabot/betabot_description/meshes/betabot_wheel.dae" />
+        <mesh filename="package://betabot_description/meshes/betabot_wheel.dae" />
       </geometry>
       <material name="">
@@ -102,5 +108,5 @@
       <geometry>
         <mesh
-          filename="package://betabot/betabot_description/meshes/betabot_wheel.dae" />
+          filename="package://betabot_description/meshes/betabot_wheel.dae" />
       </geometry>
     </collision> -->
@@ -120,5 +126,5 @@
   </joint>
 <!-- ***** BETABOT FRONT CASTER WHEEL ***** -->
-  <!-- LINK -->
+   <!-- LINK -->
   <link name="front_caster_link">
     <inertial>
@@ -130,5 +136,5 @@
       <origin xyz="0 0 0" rpy="0 0 0" />
       <geometry>
-        <mesh filename="package://betabot/betabot_description/meshes/betabot_caster.dae" />
+        <mesh filename="package://betabot_description/meshes/betabot_caster.dae" />
       </geometry>
       <material name="">
@@ -142,5 +148,5 @@
       <geometry>
         <mesh
-          filename="package://betabot/betabot_description/meshes/betabot_caster.dae" />
+          filename="package://betabot_description/meshes/betabot_caster.dae" />
       </geometry>
     </collision> -->
@@ -170,5 +176,5 @@
       <origin xyz="0 0 0" rpy="0 0 0" />
       <geometry>
-        <mesh filename="package://betabot/betabot_description/meshes/betabot_caster.dae" />
+        <mesh filename="package://betabot_description/meshes/betabot_caster.dae" />
       </geometry>
       <material
@@ -183,5 +189,5 @@
       <geometry>
         <mesh
-          filename="package://betabot/betabot_description/meshes/betabot_caster.dae" />
+          filename="package://betabot_description/meshes/betabot_caster.dae" />
       </geometry>
     </collision> -->
@@ -206,5 +212,5 @@
       <origin xyz="0 0 0" rpy="0 1.570 0" />
       <geometry>
-        <mesh filename="package://betabot/betabot_description/meshes/raspicam.dae" />
+        <mesh filename="package://betabot_description/meshes/raspicam.dae" />
       </geometry>
         <material name="">
@@ -238,5 +244,5 @@
       <origin xyz="0 0 -0.032" rpy="0 0 0"/>
       <geometry>
-        <mesh filename="package://betabot/betabot_description/meshes/rplidar.dae"/>
+        <mesh filename="package://betabot_description/meshes/rplidar.dae"/>
       </geometry>
     </visual>
@@ -253,4 +259,30 @@
     <parent link="base_link"/>
     <child link="rplidar_link"/>
-  </joint>]0i0
+  </joint>
+<!-- ***** IMU SENSOR PART ***** -->
+  <link name="imu_sensor_link">
+      <collision>
+          <origin xyz="0 0 0" rpy="0 0 0"/>
+          <geometry>
+              <box size="0.02 0.02 0.02"/>
+          </geometry>
+      </collision>
+      <visual>
+          <origin xyz="0 0 0" rpy="0 0 0"/>
+          <geometry>
+              <box size="0.02 0.02 0.02"/>
+          </geometry>
+      </visual>
+      <inertial>
+          <mass value="0.001" />
+          <origin xyz="0 0 0" rpy="0 0 0"/>
+          <inertia ixx="0.00000015" ixy="0" ixz="0" iyy="0.00000015" iyz="0" izz="0.00000015" />
+      </inertial>
+  </link>
+  <joint name="imu_sensor_joint" type="fixed">
+      <axis xyz="0 0 1" />
+      <origin xyz="0 0 0" rpy="0 0 0"/>
+      <parent link="base_link"/>
+      <child link="imu_sensor_link"/>
+  </joint>
 </robot>

Commit message: fixed links-joints coordinates and their collision also add rplidar a2 link

File: betabot_description/urdf/betabot.urdf.xacro (robot description, xacro)
@@ -9,5 +9,5 @@
 <robot name="betabot" xmlns:xacro="http://www.ros.org/wiki/xacro">
 <!-- CALL HEADER FILES FOR MACROS AND GAZEBO PLUGINS -->
-  <xacro:include filename="$(find betabot_description)/urdf/betabot.gazebo" />
+  <xacro:include filename="$(find betabot_description)/urdf/betabot.gazebo.xacro" />
   <xacro:include filename="$(find betabot_description)/urdf/materials.xacro" />
   <xacro:include filename="$(find betabot_description)/urdf/macros.xacro" />
@@ -46,9 +46,9 @@
         <cylinder length="0.004" radius="0.15"/>
       </geometry>
-      <origin rpy="0 0 0" xyz="0  0 0.0825"/>
-    </collision>
-  </link>
-<!-- ***** BETABOT LEFT WHEEL PART ***** -->
-  <link name="left_wheel_link">
+      <origin rpy="0 0 0" xyz="0  0 0.05"/>
+    </collision>
+  </link>
+<!-- ***** BETABOT RIGHT WHEEL PART ***** -->
+  <link name="right_wheel_link">
     <inertial>
       <origin xyz="1.7347E-17 -7.3726E-17 -0.015" rpy="0 0 0" />
@@ -73,31 +73,71 @@
     <collision>
       <geometry>
-        <cylinder length="0.025" radius="0.0325"/>
-      </geometry>
-      <origin rpy="0 0 0" xyz="0 0 -0.02"/>
+        <cylinder length="0.03" radius="0.0325"/>
+      </geometry>
+      <origin rpy="0 0 0" xyz="0 0 0.016"/>
+    </collision>
+  </link>
+  <!-- JOINT -->
+  <joint name="right_wheel_joint" type="continuous">
+    <origin xyz="0 -0.097 -0.0125" rpy="-1.5708 1.3735 3.14159265359" />
+    <parent link="base_link" />
+    <child link="right_wheel_link" />
+    <axis xyz="0 0 -1" />
+  </joint>
+<!-- ***** BETABOT LEFT WHEEL PART ***** -->
+  <!-- LINK -->
+  <link name="left_wheel_link">
+    <inertial>
+      <origin xyz="-1.7347E-17 -7.3726E-17 -0.015" rpy="0 0 0" />
+      <mass value="0.5" />
+      <inertia ixx="0.001" ixy="0.0" ixz="0.0" iyy="0.001" iyz="0.0" izz="0.001" />
+    </inertial>
+    <visual>
+      <origin xyz="0 0 0" rpy="0 0 0" />
+      <geometry>
+        <mesh filename="package://betabot_description/meshes/betabot_wheel.dae" />
+      </geometry>
+      <material name="">
+        <color rgba="0.79216 0.81961 0.93333 1" />
+      </material>
+    </visual>
+    <!-- <collision>
+      <origin
+        xyz="0 0 0"
+        rpy="0 0 0" />
+      <geometry>
+        <mesh
+          filename="package://betabot_description/meshes/betabot_wheel.dae" />
+      </geometry>
+    </collision> -->
+    <collision>
+      <geometry>
+        <cylinder length="0.03" radius="0.0325"/>
+      </geometry>
+      <origin rpy="0 0 0" xyz="0 0 0.016"/>
     </collision>
   </link>
   <!-- JOINT -->
   <joint name="left_wheel_joint" type="continuous">
-    <origin xyz="-0.095 0 -0.0125" rpy="-1.5708 1.3735 -1.5708" />
+    <origin xyz="0 0.097 -0.0125" rpy="-1.5708 1.5228 0" />
     <parent link="base_link" />
     <child link="left_wheel_link" />
     <axis xyz="0 0 1" />
   </joint>
-<!-- ***** BETABOT RIGHT WHEEL PART ***** -->
-  <!-- LINK -->
-  <link name="right_wheel_link">
-    <inertial>
-      <origin xyz="-1.7347E-17 -7.3726E-17 -0.015" rpy="0 0 0" />
-      <mass value="0.5" />
-      <inertia ixx="0.001" ixy="0.0" ixz="0.0" iyy="0.001" iyz="0.0" izz="0.001" />
-    </inertial>
-    <visual>
-      <origin xyz="0 0 0" rpy="0 0 0" />
-      <geometry>
-        <mesh filename="package://betabot_description/meshes/betabot_wheel.dae" />
+<!-- ***** BETABOT FRONT CASTER WHEEL ***** -->
+   <!-- LINK -->
+  <link name="front_caster_link">
+    <inertial>
+      <origin xyz="0 -0.011704 0.02" rpy="0 0 0" />
+      <mass value="0.2" />
+      <inertia ixx="0.001" ixy="0.0" ixz="0.0" iyy="0.001" iyz="0.0"  izz="0.001" />
+    </inertial>
+    <visual>
+      <origin xyz="0 0 0" rpy="0 0 0" />
+      <geometry>
+        <mesh filename="package://betabot_description/meshes/betabot_caster.dae" />
       </geometry>
       <material name="">
-        <color rgba="0.79216 0.81961 0.93333 1" />
+        <color rgba="0.65098 0.61961 0.58824 1" />
       </material>
     </visual>
@@ -108,28 +148,28 @@
       <geometry>
         <mesh
-          filename="package://betabot_description/meshes/betabot_wheel.dae" />
-      </geometry>
-    </collision> -->
-    <collision>
-      <geometry>
-        <cylinder length="0.025" radius="0.0325"/>
-      </geometry>
-      <origin rpy="0 0 0" xyz="0  0 -0.02"/>
-    </collision>
-  </link>
-  <!-- JOINT -->
-  <joint name="right_wheel_joint" type="continuous">
-    <origin xyz="0.095 0 -0.0125" rpy="-1.5708 1.5228 1.5708" />
+          filename="package://betabot_description/meshes/betabot_caster.dae" />
+      </geometry>
+    </collision> -->
+    <collision>
+      <geometry>
+         <sphere radius="0.020"/>
+      </geometry>
+      <origin rpy="0 0 0" xyz="0 -0.0026 0"/>
+    </collision>
+  </link>
+  <!-- JOINT -->
+  <joint name="front_caster_joint" type="fixed">
+    <origin xyz="0.105 0 -0.02231" rpy="1.5708 6.123E-17 1.5708" />
     <parent link="base_link" />
-    <child link="right_wheel_link" />
-    <axis xyz="0 0 -1" />
-  </joint>
-<!-- ***** BETABOT FRONT CASTER WHEEL ***** -->
-   <!-- LINK -->
-  <link name="front_caster_link">
-    <inertial>
-      <origin xyz="0 -0.011704 0.02" rpy="0 0 0" />
+    <child link="front_caster_link" />
+    <axis xyz="0 0 0" />
+  </joint>
+<!-- ***** BETABOT BACK CASTER WHEEL ***** -->
+  <!-- LINK -->
+  <link name="back_caster_link">
+    <inertial>
+      <origin xyz="0 0.011704 0.02" rpy="0 0 0" />
       <mass value="0.2" />
-      <inertia ixx="0.001" ixy="0.0" ixz="0.0" iyy="0.001" iyz="0.0"  izz="0.001" />
+      <inertia ixx="0.001" ixy="0.0" ixz="0.0" iyy="0.001" iyz="0.0" izz="0.001" />
     </inertial>
     <visual>
@@ -138,5 +178,6 @@
         <mesh filename="package://betabot_description/meshes/betabot_caster.dae" />
       </geometry>
-      <material name="">
+      <material
+        name="">
         <color rgba="0.65098 0.61961 0.58824 1" />
       </material>
@@ -155,51 +196,10 @@
          <sphere radius="0.020"/>
       </geometry>
-      <origin rpy="0 0 0" xyz="0 0 0"/>
-    </collision>
-  </link>
-  <!-- JOINT -->
-  <joint name="front_caster_joint" type="fixed">
-    <origin xyz="0 -0.105 -0.02231" rpy="1.5708 6.123E-17 1.5708" />
-    <parent link="base_link" />
-    <child link="front_caster_link" />
-    <axis xyz="0 0 0" />
-  </joint>
-<!-- ***** BETABOT BACK CASTER WHEEL ***** -->
-  <!-- LINK -->
-  <link name="back_caster_link">
-    <inertial>
-      <origin xyz="0 0.011704 0.02" rpy="0 0 0" />
-      <mass value="0.2" />
-      <inertia ixx="0.001" ixy="0.0" ixz="0.0" iyy="0.001" iyz="0.0" izz="0.001" />
-    </inertial>
-    <visual>
-      <origin xyz="0 0 0" rpy="0 0 0" />
-      <geometry>
-        <mesh filename="package://betabot_description/meshes/betabot_caster.dae" />
-      </geometry>
-      <material
-        name="">
-        <color rgba="0.65098 0.61961 0.58824 1" />
-      </material>
-    </visual>
-    <!-- <collision>
-      <origin
-        xyz="0 0 0"
-        rpy="0 0 0" />
-      <geometry>
-        <mesh
-          filename="package://betabot_description/meshes/betabot_caster.dae" />
-      </geometry>
-    </collision> -->
-    <collision>
-      <geometry>
-         <sphere radius="0.020"/>
-      </geometry>
-      <origin rpy="0 0 0" xyz="0 -0.002 0"/>
+      <origin rpy="0 0 0" xyz="0 -0.0026 0"/>
     </collision>
   </link>
   <!-- JOINT -->
   <joint name="back_caster_joint" type="fixed">
-    <origin xyz="0 0.105 -0.02231" rpy="1.5708 6.123E-17 1.5708" />
+    <origin xyz="-0.105 0 -0.02231" rpy="1.5708 6.123E-17 1.5708" />
     <parent link="base_link" />
     <child link="back_caster_link" />
@@ -210,5 +210,5 @@
   <link name="camera_link">
     <visual>
-      <origin xyz="0 0 0" rpy="0 1.570 0" />
+      <origin xyz="0 0 0" rpy="0 1.570 1.570" />
       <geometry>
         <mesh filename="package://betabot_description/meshes/raspicam.dae" />
@@ -228,37 +228,10 @@
   <joint name="camera_joint" type="fixed">
     <axis xyz="0 0 0" />
-    <origin xyz="0 -0.148 0.040" rpy="0 0 -1.570"/>
+    <origin xyz="0.148 0 0.036" rpy="0 0 0"/>
     <parent link="base_link"/>
     <child link="camera_link"/>
   </joint>
-<!-- ***** RPLiDAR A1 RANGE FINDER SENSOR SIMULATED PART ***** -->
-  <!-- LINK -->
-  <link name="rplidar_link">
-    <collision>
-      <origin xyz="0 0 0" rpy="0 0 0"/>
-      <geometry>
-        <box size="0.1 0.1 0.1"/>
-      </geometry>
-    </collision>
-    <visual>
-      <origin xyz="0 0 -0.032" rpy="0 0 0"/>
-      <geometry>
-        <mesh filename="package://betabot_description/meshes/rplidar.dae"/>
-      </geometry>
-    </visual>
-    <inertial>
-      <mass value="1e-5" />
-      <origin xyz="0 0 0" rpy="0 0 0"/>
-      <inertia ixx="1e-6" ixy="0" ixz="0" iyy="1e-6" iyz="0" izz="1e-6" />
-    </inertial>
-  </link>
-  <!-- JOINT -->
-  <joint name="rplidar_joint" type="fixed">
-    <axis xyz="0 1 0" />
-    <origin xyz="0 0 .1" rpy="0 0 0"/>
-    <parent link="base_link"/>
-    <child link="rplidar_link"/>
-  </joint>
 <!-- ***** IMU SENSOR PART ***** -->
+  <!-- LINK -->
   <link name="imu_sensor_link">
       <collision>
@@ -280,4 +253,5 @@
       </inertial>
   </link>
+  <!-- JOINT -->
   <joint name="imu_sensor_joint" type="fixed">
       <axis xyz="0 0 1" />
@@ -286,3 +260,59 @@
       <child link="imu_sensor_link"/>
   </joint>
+<!-- ***** RPLiDAR A1 RANGE FINDER SENSOR SIMULATED PART ***** -->
+  <!-- LINK -->
+  <!-- <link name="rplidar_link">
+    <collision>
+      <origin xyz="0 0 -0.03" rpy="0 0 0"/>
+      <geometry>
+         <sphere radius="0.045"/>
+      </geometry>
+    </collision>
+    <visual>
+      <origin xyz="0 0 -0.032" rpy="0 0 0"/>
+      <geometry>
+        <mesh filename="package://betabot_description/meshes/rplidar.dae"/>
+      </geometry>
+    </visual>
+    <inertial>
+      <mass value="1e-5" />
+      <origin xyz="0 0 0" rpy="0 0 0"/>
+      <inertia ixx="1e-6" ixy="0" ixz="0" iyy="1e-6" iyz="0" izz="1e-6" />
+    </inertial>
+  </link> -->
+  <!-- JOINT -->
+  <!-- <joint name="rplidar_joint" type="fixed">
+    <axis xyz="0 1 0" />
+    <origin xyz="0 0 .1" rpy="0 0 0"/>
+    <parent link="base_link"/>
+    <child link="rplidar_link"/>
+  </joint> -->
+<!-- ***** RPLiDAR A2 RANGE FINDER SENSOR SIMULATED PART ***** -->
+  <!-- LINK -->
+  <link name="rplidar_link">
+    <collision>
+      <origin xyz="0 0 -0.03" rpy="0 0 0"/>
+      <geometry>
+         <sphere radius="0.045"/>
+      </geometry>
+    </collision>
+    <visual>
+      <origin xyz="0 0 -0.032" rpy="0 0 0"/>
+      <geometry>
+        <mesh filename="package://betabot_description/meshes/rplidar_a2.dae"/>
+      </geometry>
+    </visual>
+    <inertial>
+      <mass value="1e-5" />
+      <origin xyz="0 0 0" rpy="0 0 0"/>
+      <inertia ixx="1e-6" ixy="0" ixz="0" iyy="1e-6" iyz="0" izz="1e-6" />
+    </inertial>
+  </link>
+  <!-- JOINT -->
+  <joint name="rplidar_joint" type="fixed">
+    <axis xyz="0 1 0" />
+    <origin xyz="0 0 .109" rpy="0 0 0"/>
+    <parent link="base_link"/>
+    <child link="rplidar_link"/>
+  </joint>
 </robot>

Commit message: clean worlds launch files

File: betabot_description/urdf/betabot.urdf.xacro (robot description, xacro)
@@ -166,5 +166,5 @@
     <child link="front_caster_link" />
     <axis xyz="0 0 0" />
-    <dynamics damping="0.0" friction="0.0"/>
+    <dynamics damping="0.1" friction="0.1"/>
   </joint>
 <!-- ***** BETABOT BACK CASTER WHEEL ***** -->
@@ -208,5 +208,5 @@
     <child link="back_caster_link" />
     <axis xyz="0 0 0" />
-    <dynamics damping="0.0" friction="0.0"/>
+    <dynamics damping="0.1" friction="0.1"/>
   </joint>
 <!-- ***** BETABOT EXTENSION ***** -->

Commit message: fix LiDAR pose

File: betabot_description/urdf/betabot.urdf.xacro (robot description, xacro)
@@ -360,5 +360,5 @@
   <joint name="rplidar_joint" type="fixed">
     <axis xyz="0 1 0" />
-    <origin xyz="0 0 .109" rpy="0 0 1.57"/>
+    <origin xyz="0 0 .109" rpy="0 0 0"/>
     <parent link="base_link"/>
     <child link="rplidar_link"/>
